File: PCB/TS65.kicad_pcb (KiCad board)
At the start: 2 copper layers, 299.2 x 112.1 mm, 419 parts, among them P1 USB_TYPE_C, P2 USB3_AFEMALE, P3 CONN_17, Q1 3.3V REG IC, U1 MK20DX256VLH7, U2 IS31FL3731, X1 CRYSTAL

Commit message: PCB version 0.3
Case still to be updated to Rev 0.3
Parts:
- removed LEDG10, LEDG11, LEDG12, LEDG13, LEDG14, LEDG15, LEDG16, LEDG9, LEDGR11, LEDGR12, LEDGR13, LEDGR14, LEDGR15, LEDGR16, LEDGR17, LEDGR18: LED, prettylib:LED_1206
- added C10: 0.1 uF, prettylib:SMD_0805, B.Cu at (167.7, 93.5)
- added C11: 0.1 uF, prettylib:SMD_0805, B.Cu at (136.6, 96.1)
- added C12: 0.1 uF, prettylib:SMD_0805, B.Cu at (104.1, 95.7)
- added C13: 0.1 uF, prettylib:SMD_0805, B.Cu at (72.7, 95.3)
- added C14: 0.1 uF, prettylib:SMD_0805, B.Cu at (63.3, 154.5)
- added C15: 0.1 uF, prettylib:SMD_0805, B.Cu at (95.1, 151.9)
- added C16: 0.1 uF, prettylib:SMD_0805, B.Cu at (127.2, 153.8)
- added C17: 0.1 uF, prettylib:SMD_0805, B.Cu at (167.0, 150.6)
- added C18: 0.1uF, prettylib:SMD_0805, B.Cu at (115.7, 65.6)
- added C19: 10uF, prettylib:SMD_0805, B.Cu at (144.6, 70.6)
- added CR10: 0.1 uF, prettylib:SMD_0805, B.Cu at (197.9, 96.6)
- added CR11: 0.1 uF, prettylib:SMD_0805, B.Cu at (233.3, 96.0)
- added CR12: 0.1 uF, prettylib:SMD_0805, B.Cu at (267.6, 95.4)
- added CR13: 0.1 uF, prettylib:SMD_0805, B.Cu at (303.2, 96.9)
- added CR14: 0.1 uF, prettylib:SMD_0805, B.Cu at (337.7, 96.2)
- added CR15: 0.1 uF, prettylib:SMD_0805, B.Cu at (338.6, 152.4)
- added CR16: 0.1 uF, prettylib:SMD_0805, B.Cu at (317.3, 152.3)
- added CR17: 0.1 uF, prettylib:SMD_0805, B.Cu at (284.3, 152.1)
- added CR18: 0.1 uF, prettylib:SMD_0805, B.Cu at (251.4, 152.4)
- added CR19: 0.1 uF, prettylib:SMD_0805, B.Cu at (220.0, 151.6)
- added CR20: 0.1uF, prettylib:SMD_0805, B.Cu at (249.1, 65.5)
- added CR21: 10uF, prettylib:SMD_0805, B.Cu at (279.6, 71.4)
- added F1: PTC FUSE, prettylib:Fuse_SMD1206_HandSoldering, B.Cu at (153.5, 63.0)
- added FR1: PTC FUSE, prettylib:Fuse_SMD1206_HandSoldering, B.Cu at (288.5, 62.5)
- added LEDI1: LED, prettylib:LED-3MM, B.Cu at (337.0, 71.0)
- added LEDI2: LED, prettylib:LED-3MM, B.Cu at (330.0, 71.0)
- added LEDI3: LED, prettylib:LED-3MM, B.Cu at (323.0, 71.0)
- added P4: FLASH_HDR, prettylib:JLINK_NEEDLE, B.Cu at (145.0, 116.0)
- added PR4: FLASH_HDR, prettylib:JLINK_NEEDLE, B.Cu at (247.7, 134.6)
- added R13: 330, prettylib:SMD_0805, B.Cu at (139.7, 72.6)
- added RR13: 330, prettylib:SMD_0805, B.Cu at (271.8, 72.4)
- added U3: 74HCT1G125, prettylib:SOT-753, B.Cu at (135.5, 72.5)
- added U4: IP4234CZ6, prettylib:SOT457, B.Cu at (156.9, 73.2)
- added UR3: 74HCT1G125, prettylib:SOT-753, B.Cu at (268.0, 72.3)
- added UR4: IP4234CZ6, prettylib:SOT457, B.Cu at (291.7, 72.9)
- BREAKHOLES1, BREAKHOLES2: value BreakHoles -> MISC
- FID1, FID2, FID3, FID4, HOLE1: value (none) -> MISC
- FIDR1: renamed from FID1; value (none) -> MISC
- FIDR2: renamed from FID2; value (none) -> MISC
- FIDR3: renamed from FID3; value (none) -> MISC
- FIDR4: renamed from FID4; value (none) -> MISC
- HOLER1: renamed from HOLE1; value (none) -> MISC
- LEDD1, LEDDR1: footprint prettylib:LED_1206 -> prettylib:LED_0805
- LEDG1, LEDG2, LEDG3, LEDG4, LEDG5, LEDG6, LEDG7, LEDG8, LEDGR1, LEDGR10, LEDGR2, LEDGR3, LEDGR4, LEDGR5, LEDGR6, LEDGR7, LEDGR8, LEDGR9: value LED -> WS2812B; footprint prettylib:LED_1206 -> prettylib:WS2812B
- LOGO1, LOGO2: value LOGO -> MISC
- LOGO3, LOGO4: value OSHW -> MISC
- LOGOR1: renamed from LOGO1; value LOGO -> MISC
- LOGOR2: renamed from LOGO2; value LOGO -> MISC
- LOGOR3, LOGOR4: renamed from LOGO3; value OSHW -> MISC
- P3, PR3: value CONN_17 -> CONN_15; footprint prettylib:HEADER_1x17 -> prettylib:HEADER_1x15
- S1, S10, S11, S12, S13, S14, S15, S16, S17, S18, S19, S19_2, S2, S20, S21, S22, S23, S24, S25, S26, S26_2, S27, S27_2, S27_3, S27_4, S28, S28_2, S28_3, S28_4, S28_5, S28_6, S28_7, S29, S29_2, S29_3, S29_4, S3, S30, S30_2, S30_3, S31, S31_2, S4, S5, S6, S7, S8, S9, SR1, SR10, SR11, SR12, SR13, SR14, SR15, SR16, SR17, SR18, SR19, SR2, SR20, SR21, SR22, SR23, SR24, SR24_2, SR25, SR26, SR27, SR28, SR29, SR3, SR30, SR30_2, SR31, SR32, SR33, SR33_2, SR34, SR34_2, SR35_3, SR36_2, SR36_3, SR36_4, SR36_5, SR37, SR37_2, SR37_3, SR37_4, SR37_5, SR37_6, SR37_7, SR38, SR38_2, SR38_3, SR39, SR4, SR40, SR41, SR41_2, SR41_3, SR42, SR5, SR6, SR7, SR8, SR9: footprint prettylib:MXALPS -> prettylib:MXALPS2
- STAB1, STAB3, STAB5, STABR2: value MX_225 -> MISC; footprint prettylib:MX_225 -> prettylib:MX_200
- STAB2, STABR1, STABR7: value MX_275 -> MISC; footprint prettylib:MX_275 -> prettylib:MX_200
- STAB4, STABR4: value MX_225_Plated -> MISC; footprint prettylib:MX_225 -> prettylib:MX_200
- STABR3, STABR5: value MX_200 -> MISC
- STABR6: value MX_275_Plated -> MISC; footprint prettylib:MX_275 -> prettylib:MX_200
- moved LEDGR7 127.9 mm to (311.5, 152.5)
- moved LEDG5 115.7 mm to (70.0, 152.0), turned to 180 degrees
- moved LEDGR10 91.0 mm to (214.0, 152.5)
- moved LEDG1 84.9 mm to (163.0, 96.0)
- moved LEDGR8 79.4 mm to (280.0, 152.0), turned to 90 degrees
- moved LOGOR3 76.3 mm to (271.0, 133.9)
- moved LOGOR4 76.3 mm to (271.0, 133.9)
- moved LOGOR1 74.5 mm to (290.0, 133.9)
- moved LOGOR2 74.5 mm to (290.0, 133.9)
- moved LEDGR5 65.1 mm to (343.0, 96.0), turned to 180 degrees
- moved LEDG2 63.9 mm to (131.0, 96.0), turned to 0 degrees
- moved LEDG7 63.4 mm to (133.0, 152.0), turned to 180 degrees
- moved LEDGR9 59.5 mm to (246.5, 152.5)
- moved LEDGR4 58.3 mm to (309.5, 99.0), turned to 270 degrees
- moved LEDG6 58.0 mm to (100.0, 152.0), turned to 270 degrees
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Connections:
- net /mcu/RX0 renamed /mcu/UART0-
- net /mcu/RX1 renamed /mcu/UART1-
- net /mcu/RX2 renamed /mcu/UART2-
- net /mcu/TX0 renamed /mcu/UART0+
- net /mcu/TX1 renamed /mcu/UART1+
- net /mcu/TX2 renamed /mcu/UART2+
- net /mcu/USB_DM renamed /mcu/USB_D-
- net /mcu/USB_DP renamed /mcu/USB_D+
- net /mcuR/GNDR renamed /mcuR/GND
- net /mcuR/RX0 renamed /mcuR/UART0-
- net /mcuR/RX1 renamed /mcuR/UART1-
- net /mcuR/RX2 renamed /mcuR/UART2-
- net /mcuR/TX0 renamed /mcuR/UART0+
- net /mcuR/TX1 renamed /mcuR/UART1+
- net /mcuR/TX2 renamed /mcuR/UART2+
- net /mcuR/USB_DM renamed /mcuR/USB_D-
- net /mcuR/USB_DP renamed /mcuR/USB_D+
- LEDG1 pad 1: /ledmatrix/CA1 -> +5V
- LEDG1 pad 2: /ledmatrix/CA6 -> Net-(LEDG1-Pad2)
- LEDG2 pad 1: /ledmatrix/CA2 -> +5V
- LEDG2 pad 2: /ledmatrix/CA3 -> Net-(LEDG2-Pad2)
- LEDG3 pad 1: /ledmatrix/CA2 -> +5V
- LEDG3 pad 2: /ledmatrix/CA6 -> Net-(LEDG3-Pad2)
- LEDG4 pad 1: /ledmatrix/CA3 -> +5V
- LEDG4 pad 2: /ledmatrix/CA6 -> Net-(LEDG4-Pad2)
- LEDG5 pad 1: /ledmatrix/CA4 -> +5V
- LEDG5 pad 2: /ledmatrix/CA6 -> Net-(LEDG5-Pad2)
- LEDG6 pad 1: /ledmatrix/CA6 -> +5V
- LEDG6 pad 2: /ledmatrix/CA1 -> Net-(LEDG6-Pad2)
- LEDG7 pad 1: /ledmatrix/CA6 -> +5V
- LEDG7 pad 2: /ledmatrix/CA2 -> Net-(LEDG7-Pad2)
- LEDG8 pad 1: /ledmatrix/CA5 -> +5V
- LEDG8 pad 2: /ledmatrix/CA6 -> Net-(LEDG8-Pad2)
- LEDGR1 pad 1: /ledmatrixR/CA2 -> +5V
- LEDGR1 pad 2: /ledmatrixR/CA6 -> Net-(LEDGR1-Pad2)
- LEDGR10 pad 1: /ledmatrixR/CA4 -> +5V
- LEDGR10 pad 2: /ledmatrixR/CA7 -> Net-(LEDGR10-Pad2)
- LEDGR2 pad 1: /ledmatrixR/CA3 -> +5V
- LEDGR2 pad 2: /ledmatrixR/CA6 -> Net-(LEDGR2-Pad2)
- LEDGR3 pad 1: /ledmatrixR/CA4 -> +5V
- LEDGR3 pad 2: /ledmatrixR/CA6 -> Net-(LEDGR3-Pad2)
- LEDGR4 pad 1: /ledmatrixR/CA5 -> +5V
- LEDGR4 pad 2: /ledmatrixR/CA6 -> Net-(LEDGR4-Pad2)
- LEDGR5 pad 1: /ledmatrixR/CA7 -> +5V
- LEDGR5 pad 2: /ledmatrixR/CA6 -> Net-(LEDGR5-Pad2)
- LEDGR6 pad 1: /ledmatrixR/CA8 -> +5V
- LEDGR6 pad 2: /ledmatrixR/CA6 -> Net-(LEDGR6-Pad2)
- LEDGR7 pad 1: /ledmatrixR/CA1 -> +5V
- LEDGR7 pad 2: /ledmatrixR/CA7 -> Net-(LEDGR7-Pad2)
- LEDGR8 pad 1: /ledmatrixR/CA2 -> +5V
- LEDGR8 pad 2: /ledmatrixR/CA7 -> Net-(LEDGR8-Pad2)
- LEDGR9 pad 1: /ledmatrixR/CA3 -> +5V
- LEDGR9 pad 2: /ledmatrixR/CA7 -> Net-(LEDGR10-Pad4)
- P1 pad A4: +5V -> /mcu/VBUS
- P1 pad A6: Net-(P1-PadA6) -> /mcu/USB_D_IN+
- P1 pad A7: Net-(P1-PadA7) -> /mcu/USB_D_IN-
- P1 pad A9: +5V -> /mcu/VBUS
- P1 pad B4: +5V -> /mcu/VBUS
- P1 pad B6: Net-(P1-PadA6) -> /mcu/USB_D_IN+
- P1 pad B7: Net-(P1-PadA7) -> /mcu/USB_D_IN-
- P1 pad B9: +5V -> /mcu/VBUS
- P2 pad 1: +5V -> /mcu/VBUS
- P3 pad 2: /mcu/SWD_DIO -> VSS
- P3 pad 3: VSS -> /mcu/SWD_DIO
- PR1 pad A4: +5V -> /mcuR/VBUS
- PR1 pad A6: Net-(PR1-PadA6) -> /mcuR/USB_D_IN+
- PR1 pad A7: Net-(PR1-PadA7) -> /mcuR/USB_D_IN-
- PR1 pad A9: +5V -> /mcuR/VBUS
- PR1 pad B4: +5V -> /mcuR/VBUS
- PR1 pad B6: Net-(PR1-PadA6) -> /mcuR/USB_D_IN+
- PR1 pad B7: Net-(PR1-PadA7) -> /mcuR/USB_D_IN-
- PR1 pad B9: +5V -> /mcuR/VBUS
- PR2 pad 1: +5V -> /mcuR/VBUS
- PR3 pad 2: /mcuR/SWD_DIO -> VSS
- PR3 pad 3: VSS -> /mcuR/SWD_DIO
- R1 pad 1: Net-(P1-PadA7) -> Net-(R1-Pad1)
- R2 pad 1: Net-(P1-PadA6) -> Net-(R2-Pad1)
- RR1 pad 1: Net-(PR1-PadA7) -> Net-(RR1-Pad1)
- RR2 pad 1: Net-(PR1-PadA6) -> Net-(RR2-Pad1)
- S19_2 pad 1: Net-(D19-Pad1) -> /mcu/PTD0
- S19_2 pad 2: /mcu/PTD0 -> Net-(D19-Pad1)
Routing:
- net VSS: track 650.5 -> 1409.9 mm, vias 25 -> 36
- net +5V: track 324.6 -> 945.7 mm, vias 12 -> 21
- net /ledmatrixR/CA8: track 519.5 -> 200.2 mm, vias 11 -> 3
- net /ledmatrixR/CA7: track 507.9 -> 231.9 mm
- net /ledmatrix/CA6: track 474.3 -> 229.2 mm, vias 8 -> 2
- net /ledmatrix/CA2: track 560.3 -> 316.7 mm, vias 7 -> 5
- net /ledmatrix/CA5: track 420.8 -> 291.6 mm, vias 4 -> 5
- net /ledmatrixR/CA6: track 525.4 -> 403.4 mm, vias 11 -> 9
- net VDD: track 379.9 -> 498.6 mm, vias 6 -> 8
- net /ledmatrixR/CA3: track 505.2 -> 395.9 mm, vias 8 -> 3
- net /ledmatrix/CA8: track 394.1 -> 290.2 mm, vias 3 -> 1
- net /ledmatrix/CA7: track 261.4 -> 163.7 mm, vias 1 -> 0
- net Net-(LEDGR1-Pad4): track 0.00 -> 93.6 mm, vias 0 -> 2
- net /mcuR/PTA5: track 4.60 -> 89.3 mm, vias 0 -> 4
- net /ledmatrixR/CA5: track 483.5 -> 401.0 mm, vias 7 -> 3
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Other:
- board text added: "3.3V VSS 5V RX0 TX0 RX1 TX1 AUD SDA0 SCL0"
- board text added: "DIO"
- board text added: "RST"
- board text added: "TS65-L Rev 0.3 Designed & Drawn in KiCAD by Mohit 'MOZ' Garg"
- board text added: "TS65-R Rev 0.3 Designed & Drawn in KiCAD by Mohit 'MOZ' Garg"
- board text removed: "3.3V DIO 5V RX0 TX0 RX1 TX1 SDA0 SCL0 RST AUD"
- board text removed: "TS65-L Rev 0.2 Designed & Drawn in KiCAD by by Mohit 'MOZ' Garg Based on ICED-L Rev 1.1d"
- board text removed: "TS65-R Rev 0.2 Designed & Drawn in KiCAD by by Mohit 'MOZ' Garg Based on ICED-L Rev 1.1d"
- board text removed: "VSS"
